File: KiCAD/General_8th_MFB_LPF/General_8th_MFB_LPF.sch (KiCad schematic (older format))
At the start: 42 parts, among them J1 IN, J2 Dual_PWR_IN, J3 SGL_PWR_IN, J4 PWR_OUT, J5 OUT, U1 NJM4580, U2 NJM4580, U3 TLE2426xLP

Commit message: PCB
Parts:
- removed C13: 100u, symbol Device:CP
- removed J4: PWR_OUT, symbol Connector_Generic:Conn_01x03
- removed JP1: VCC_SEL, symbol Jumper:Jumper_3_Open
- removed JP2: GND_SEL, symbol Jumper:Jumper_3_Open
- removed JP3: VEE_SEL, symbol Jumper:Jumper_3_Open
- removed U3: TLE2426xLP, symbol Reference_Voltage:TLE2426xLP
- added C15: 100u, Capacitor_THT:CP_Radial_D6.3mm_P2.50mm, symbol Device:CP
- added C16: 0.1u, Capacitor_THT:C_Disc_D3.4mm_W2.1mm_P2.50mm, symbol Device:C
- added H1, H2, H3, H4: MountingHole, MountingHole:MountingHole_3.2mm_M3, symbol Mechanical:MountingHole
- added J5: SGL_PWR_IN, Connector_JST:JST_XH_B2B-XH-A_1x02_P2.50mm_Vertical, symbol Connector_Generic:Conn_01x02
- added J6: Dual_PWR_OUT, Connector_JST:JST_XH_B3B-XH-A_1x03_P2.50mm_Vertical, symbol Connector_Generic:Conn_01x03
- added J7: TP_GND, Connector_PinHeader_2.54mm:PinHeader_1x02_P2.54mm_Vertical, symbol Connector_Generic:Conn_01x02
- added R15, R16: 100k, Resistor_THT:R_Axial_DIN0207_L6.3mm_D2.5mm_P7.62mm_Horizontal, symbol Device:R
- added U3: NJM4580, Package_DIP:DIP-8_W7.62mm_Socket_LongPads, symbol Device:Opamp_Dual_Generic
- C1: renamed from C14; footprint (none) -> Capacitor_THT:CP_Radial_D6.3mm_P2.50mm
- C10: renamed from C8; footprint (none) -> Capacitor_THT:C_Rect_L7.0mm_W3.5mm_P2.50mm_P5.00mm
- C11: renamed from C9; footprint (none) -> Capacitor_THT:C_Disc_D3.4mm_W2.1mm_P2.50mm
- C12: renamed from C10; footprint (none) -> Capacitor_THT:C_Disc_D3.4mm_W2.1mm_P2.50mm
- C13: renamed from C11; footprint (none) -> Capacitor_THT:C_Rect_L7.0mm_W3.5mm_P2.50mm_P5.00mm
- C14: renamed from C12; footprint (none) -> Capacitor_THT:C_Rect_L7.0mm_W3.5mm_P2.50mm_P5.00mm
- C2: renamed from C15; footprint (none) -> Capacitor_THT:CP_Radial_D6.3mm_P2.50mm
- C3: renamed from C1; footprint (none) -> Capacitor_THT:C_Rect_L7.0mm_W3.5mm_P2.50mm_P5.00mm
- C4: renamed from C2; footprint (none) -> Capacitor_THT:C_Rect_L7.0mm_W3.5mm_P2.50mm_P5.00mm
- C5: renamed from C3; footprint (none) -> Capacitor_THT:C_Disc_D3.4mm_W2.1mm_P2.50mm
- C6: renamed from C4; footprint (none) -> Capacitor_THT:C_Disc_D3.4mm_W2.1mm_P2.50mm
- C7: renamed from C5; footprint (none) -> Capacitor_THT:C_Rect_L7.0mm_W3.5mm_P2.50mm_P5.00mm
- C8: renamed from C6; footprint (none) -> Capacitor_THT:C_Rect_L7.0mm_W3.5mm_P2.50mm_P5.00mm
- C9: renamed from C7; footprint (none) -> Capacitor_THT:C_Rect_L7.0mm_W3.5mm_P2.50mm_P5.00mm
- D1, D2: footprint (none) -> LED_THT:LED_D3.0mm
- J1: renamed from J2; footprint (none) -> Connector_JST:JST_XH_B3B-XH-A_1x03_P2.50mm_Vertical
- J2: renamed from J1; footprint (none) -> Connector_JST:JST_XH_B2B-XH-A_1x02_P2.50mm_Vertical
- J3: value SGL_PWR_IN -> 4TH_OUT; footprint (none) -> Connector_JST:JST_XH_B2B-XH-A_1x02_P2.50mm_Vertical
- J4: renamed from J5; value OUT -> 8TH_OUT; footprint (none) -> Connector_JST:JST_XH_B2B-XH-A_1x02_P2.50mm_Vertical
- R1: renamed from R13; footprint (none) -> Resistor_THT:R_Axial_DIN0207_L6.3mm_D2.5mm_P7.62mm_Horizontal
- R10: renamed from R8; footprint (none) -> Resistor_THT:R_Axial_DIN0207_L6.3mm_D2.5mm_P7.62mm_Horizontal
- R11: renamed from R9; footprint (none) -> Resistor_THT:R_Axial_DIN0207_L6.3mm_D2.5mm_P7.62mm_Horizontal
- R12: renamed from R10; footprint (none) -> Resistor_THT:R_Axial_DIN0207_L6.3mm_D2.5mm_P7.62mm_Horizontal
- R13: renamed from R11; footprint (none) -> Resistor_THT:R_Axial_DIN0207_L6.3mm_D2.5mm_P7.62mm_Horizontal
- R14: renamed from R12; footprint (none) -> Resistor_THT:R_Axial_DIN0207_L6.3mm_D2.5mm_P7.62mm_Horizontal
- R2: renamed from R14; footprint (none) -> Resistor_THT:R_Axial_DIN0207_L6.3mm_D2.5mm_P7.62mm_Horizontal
- R3: renamed from R1; footprint (none) -> Resistor_THT:R_Axial_DIN0207_L6.3mm_D2.5mm_P7.62mm_Horizontal
- R4: renamed from R2; footprint (none) -> Resistor_THT:R_Axial_DIN0207_L6.3mm_D2.5mm_P7.62mm_Horizontal
- R5: renamed from R3; footprint (none) -> Resistor_THT:R_Axial_DIN0207_L6.3mm_D2.5mm_P7.62mm_Horizontal
- R6: renamed from R4; footprint (none) -> Resistor_THT:R_Axial_DIN0207_L6.3mm_D2.5mm_P7.62mm_Horizontal
- R7: renamed from R5; footprint (none) -> Resistor_THT:R_Axial_DIN0207_L6.3mm_D2.5mm_P7.62mm_Horizontal
- R8: renamed from R6; footprint (none) -> Resistor_THT:R_Axial_DIN0207_L6.3mm_D2.5mm_P7.62mm_Horizontal
- R9: renamed from R7; footprint (none) -> Resistor_THT:R_Axial_DIN0207_L6.3mm_D2.5mm_P7.62mm_Horizontal
- U1, U2: footprint (none) -> Package_DIP:DIP-8_W7.62mm_Socket_LongPads
Connections:
- net GND2 is gone; now on net GND: J1.2 (Pin_2)
- net VCC1 is gone; now on an unnamed net: J3.1 (Pin_1)
- net VCC2 is gone; now on net VCC: J1.1 (Pin_1)
- net VEE1 is gone; now on net GND: J3.2 (Pin_2)
- net VEE2 is gone; now on net VEE: J1.3 (Pin_3)
- net GND: now also C1.2, C2.1, D1.1 (K), D2.2 (A), J7.1 (Pin_1), J7.2 (Pin_2)
- net VEE: now also R2.2; no longer D2.1 (K)
- new net: D2.1 (K), R2.1
- new net: C15.1, C16.2, J5.1 (Pin_1), J6.1 (Pin_1), R15.1, U3.8 (V+)
- new net: C15.2, C16.1, J5.2 (Pin_2), J6.3 (Pin_3), R16.2, U3.4 (V-), U3.5 (+)
- new net: R15.2, R16.1, U3.3 (+)
- new net: J6.2 (Pin_2), U3.1, U3.2 (-)
- new net: U3.6 (-), U3.7
Other:
- moved on the sheet: C1, C10, C11, C12, C13, C14, C2, C3, C4, C5, C6, C7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
